File: USB to RS485 convertor.kicad_pcb (KiCad board)
At the start: 2 copper layers, 86.9 x 68 mm, 32 parts, among them J1 USB, J2 UART, J3 R485, J4 RS232, U1 FT232RL, U2 MAX485E, U3 MAX232, U4 MAX232

Commit message: Add files via upload
Parts:
- added R5: 10K, Resistor_THT:R_Axial_DIN0207_L6.3mm_D2.5mm_P7.62mm_Horizontal, F.Cu at (93.1, 101.3)
- C1, C10, C11, C12, C2, C5, C6, C7, C8, C9: footprint Capacitor_THT:C_Disc_D3.0mm_W1.6mm_P2.50mm -> Capacitor_THT:C_Disc_D4.3mm_W1.9mm_P5.00mm
- C4: footprint Capacitor_THT:C_Disc_D3.0mm_W1.6mm_P2.50mm -> Capacitor_THT:C_Disc_D5.0mm_W2.5mm_P5.00mm
- J2: value UART -> UART interface
- R1, R2, R3, R4: footprint Resistor_THT:R_Axial_DIN0204_L3.6mm_D1.6mm_P5.08mm_Horizontal -> Resistor_THT:R_Axial_DIN0207_L6.3mm_D2.5mm_P7.62mm_Horizontal
- moved R2 4.49 mm to (128.7, 60.7)
- moved C2 4.12 mm to (83.2, 102.4)
- moved C3 2.84 mm to (74.1, 103.5)
- moved C1 2.36 mm to (69.9, 100.0)
- moved C5 1.74 mm to (114.4, 106.4)
- moved D1 1.73 mm to (81.1, 66.7)
- moved D2 1.73 mm to (83.7, 66.7)
- moved R3 1.73 mm to (75.6, 66.7)
- moved R4 1.73 mm to (89.5, 66.7)
- moved C11 1.61 mm to (114.0, 81.1)
- moved C8 1.45 mm to (126.6, 101.3)
- moved C10 1.40 mm to (125.6, 75.2)
- moved R1 1.32 mm to (83.2, 78.1)
- moved C7 1.30 mm to (126.6, 108.7)
- moved C9 1.05 mm to (125.6, 83.1)
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Connections:
- U3 pad 12: /U1_RXD -> Net-(U3-R1OUT)
Routing:
- net /U2_A: track 30.0 -> 45.4 mm
- net /U2_B: track 30.3 -> 40.0 mm
- net /U1_RXD: track 79.0 -> 70.5 mm
- net Net-(JP1-B): track 5.06 -> 8.78 mm
- net Net-(U3-R1OUT): track 0.00 -> 3.71 mm
- net /V-: track 126.5 -> 123.2 mm
- net Net-(U4-C2-): track 15.9 -> 18.7 mm
- net VCC: track 28.1 -> 30.7 mm
- net /V+: track 112.8 -> 110.8 mm
- net /U1-CBUS3: track 68.9 -> 67.0 mm
- net /U1-CBUS1: track 25.6 -> 27.4 mm
- net /U1-CBUS0: track 80.2 -> 81.9 mm
- net Net-(U3-C2-): track 17.4 -> 18.4 mm
- net Net-(U3-C2+): track 16.8 -> 16.2 mm
- net Net-(U4-C2+): track 15.4 -> 16.0 mm
